File: Hardware/Stereo_Audio_Codec_Breakout_WM8960.sch (EAGLE design)
At the start: 31 parts, among them J1 QWIIC, J2 AUDIO_JACK_3.5MM_SMD, U4 WM8960, Y1 24 MHz

Commit message: Breakout routed ready for proto review
Parts:
- removed C6, C7: 4.7uF, SparkFun-Capacitors:4.7UF-0603-6.3V-(10%)
- removed H1, H2, H3, H4: STAND-OFFTIGHT, SparkFun-Hardware:STAND-OFFTIGHT
- removed J4: (no value), SparkFun-Connectors:CONN_161X16_NO_SILK
- removed LOGO2: SFE_LOGO_NAME_FLAME.1_INCH, SparkFun-Aesthetics:SFE_LOGO_NAME_FLAME.1_INCH
- added AVDD, SPKVDD: JUMPER-SMT_3_1-NC_TRACE_SILK, SparkFun-Jumpers:JUMPER-SMT_3_1-NC_TRACE_SILK
- added C10: 0.1uF, SparkFun-Capacitors:0.1UF-0402T-16V-10%
- added C11: 10uF, SparkFun-Capacitors:10UF-0805-25V-10%
- added C15, C16, C17, C18: 1nF, SparkFun-Capacitors:1.0NF/1000PF-0402-25V-10%-X7R
- added C19, C20, C23, C24, C25, C26: 1.0uF, SparkFun-Capacitors:1.0UF-0402T-16V-10%
- added C21, C22, C27, C28, C29, C30: 47nF, SparkFun-Capacitors:47NF-0402_TIGHT-25V-10%-X7R
- added D1: RED, SparkFun-LED:LED-RED0603
- added FB1, FB2, FB3: 600Ω, SparkFun-Coils:FERRITE_BEAD-0805-600Ω-100MHZ
- added L1, L2, L3, L4: 220Ω, SparkFun-Coils:FERRITE_BEAD-0805-220Ω-100MHZ-2A
- added LED: JUMPER-SMT_2_NC_TRACE_SILK, SparkFun-Jumpers:JUMPER-SMT_2_NC_TRACE_SILK
- added LOGO1: SFE_LOGO_NAME_FLAMEBLANK, SparkFun-Aesthetics:SFE_LOGO_NAME_FLAMEBLANK
- added R1, R4, R6, R7, R8, R9: 100, SparkFun-Resistors:100OHM-0402-TIGHT-1/16W-1%
- added R10: 390, SparkFun-Resistors:390OHM-0603-1/10W-1%
- added R11: 240, SparkFun-Resistors:240OHM-0603-1/10W-1%
- added R5: 1k, SparkFun-Resistors:1KOHM-0402T-1/16W-1%
- added U5: LM1117, SparkFun-IC-Power:V_REG_LM1117SOT223
- C1: value 2.2uF -> 0.1uF; device SparkFun-Capacitors:2.2UF-0603-10V-20% -> SparkFun-Capacitors:0.1UF-0402T-16V-10%
- C13: device SparkFun-Capacitors:10NF-0603-50V-10% -> SparkFun-Capacitors:10NF-0402T-25V-10%
- C2: value 2.2uF -> 10uF; device SparkFun-Capacitors:2.2UF-0603-10V-20% -> SparkFun-Capacitors:10UF-0402T-6.3V-20%
- C3, C4, C5: device SparkFun-Capacitors:0.1UF-0603-25V-(+80/-20%) -> SparkFun-Capacitors:0.1UF-0402T-16V-10%
- C8, C9: device SparkFun-Capacitors:4.7UF-0603-6.3V-(10%) -> SparkFun-Capacitors:4.7UF-0402_TIGHT-6.3V-20%-X5R
- FD1, FD2, FD3, FD4: value FIDUCIAL1X2 -> FIDUCIALUFIDUCIAL; device SparkFun-Aesthetics:FIDUCIAL1X2 -> SparkFun-Aesthetics:FIDUCIALUFIDUCIAL
- J2: value AUDIO_JACK_3.5MM_SMD -> (none); device SparkFun-Connectors:AUDIO_JACK_3.5MM_SMD -> SparkFun-Connectors:CONN_14NO_SILK
- J3: device SparkFun-Connectors:CONN_161X16_NO_SILK -> SparkFun-Connectors:CONN_14NO_SILK
- R2, R3: value 4.7k -> 2.2k; device SparkFun-Resistors:4.7KOHM-0603-1/10W-1% -> SparkFun-Resistors:2.2KOHM-0402T-1/16W-1%
Connections:
- removed net 5V: C6.2, C7.2, U4.SPKVDD1, U4.SPKVDD2
- removed net ADC-DAT: U4.ADCDAT
- removed net DAC-DAT: U4.DACDAT
- removed net DAC-LRC: U4.ADCLRC/GPIO, U4.DACLRC
- removed net GND: C13.2, C3.1, C4.1, C5.1, C6.1, C7.1, C8.1, C9.1, J1.1, U4.AGND, U4.DGND, U4.GNDPADDLE, U4.SPKGND1, U4.SPKGND2, Y1.GND
- new net ADCDAT: J2.5, U4.ADCDAT
- new net ADCLRC: J2.6, U4.ADCLRC/GPIO
- new net AGND: C1.2, C10.1, C15.2, C16.2, C17.2, C18.2, C2.2, C21.2, C22.2, C27.2, C28.2, C29.2, C30.2, C8.1, C9.1, FB1.1, J2.11, J3.6, R10.1, U4.AGND, U4.GNDPADDLE
- new net AVDD: AVDD.2, C10.2, J3.10, U4.AVDD
- new net AVDD-REG: AVDD.3, C2.1, R11.2, U5.OUT
- new net DACDAT: J2.7, U4.DACDAT
- new net DACLRC: J2.8, U4.DACLRC
- new net DGND: C11.2, C13.2, C3.1, C4.1, C5.1, FB1.2, J1.1, J2.1, R5.1, U4.DGND, U4.SPKGND1, U4.SPKGND2, Y1.GND
- new net LINPUT2: J3.13, R6.1
- new net LINPUT3: J3.12, R1.1
- new net N$1: L3.1, U4.SPEAKER_RP
- new net N$13: C20.1, C21.1, R6.2
- new net N$14: C19.1, C22.1, R4.2
- new net N$15: C23.1, C27.1, R1.2
- new net N$18: C24.1, C28.1, R7.2
- new net N$19: C25.1, C29.1, R8.2
- new net N$2: AVDD.1, FB3.1
- new net N$20: C26.1, C30.1, R9.2
- new net N$25: R10.2, R11.1, U5.ADJ
- new net N$3: L4.1, U4.SPEAKER_RN
- new net N$4: L2.1, U4.SPEAKER_LP
- new net N$45: C1.1, FB2.2, U5.IN
- new net N$5: L1.1, U4.SPEAKER_LN
- new net N$6: D1.C, R5.2
- new net N$7: D1.A, LED.1
- new net RINPUT2: J2.13, R8.1
- new net RINPUT3: J2.12, R9.1
- new net SPKVDD: C11.1, J3.1, SPKVDD.2, U4.SPKVDD1, U4.SPKVDD2
- new net VIN: FB2.1, J2.10, SPKVDD.1
- net 3.3V: now also FB3.2, J2.2, LED.2, SPKVDD.3; no longer U4.AVDD
- net BCLK: now also J2.9
- net HP_L: now also J3.9
- net HP_R: now also J3.7
- net LINPUT1: now also J3.14, R4.1; no longer C1.2
- net MICBIAS: now also J3.11
- net MONO_OUT: now also J3.8
- net N$10: now also C23.2
- net N$12: now also C20.2
- net N$29: now also C19.2; no longer C1.1
- net N$30: now also C24.2; no longer C2.1
- net N$8: now also C26.2
- net N$9: now also C25.2
- net RINPUT1: now also J2.14, R7.1; no longer C2.2
- net SCL: now also J2.4
- net SDA: now also J2.3
- net SPK_LN: now also C15.1, J3.4, L1.2; no longer U4.SPEAKER_LN
- net SPK_LP: now also C16.1, J3.5, L2.2; no longer U4.SPEAKER_LP
- net SPK_RN: now also C18.1, J3.2, L4.2; no longer U4.SPEAKER_RN
- net SPK_RP: now also C17.1, J3.3, L3.2; no longer U4.SPEAKER_RP
Other:
- note added: "AVDD VREG"
- note added: "Cut LED Jumper to disable power LED"
- note added: "Headers"
- note added: "I2C Address: 0x34 (unshifted)"
- note added: "Low-pass filters 100ohm & 47nF = 33KHz"
- note added: "Power LED"
- note added: "Power Selection Jumpers"
- note added: "Qwiic"
- note added: "Supply Voltage Ranges DCVDD: 1.7-3.6V DBVDD: 1.7-3.6V AVDD: 2.7-3.6V SPKVDD: 2.7-5.5V"
- moved on the sheet: C1, C13, C2, C3, C4, C5, C8, C9, I2C, J1, R2, R3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
