File: Hardware/Production/Stereo_Audio_Codec_Breakout_WM8960-Panel.brd (EAGLE design)
At the start: 97.3 x 96 mm, 870 parts, among them J1 QWIIC, J10 QWIIC, J13 QWIIC, J16 QWIIC, J2 QWIIC, J7 QWIIC, U1 WM8960, U10 XC6222B331MR-G, U11 WM8960, U12 XC6222B331MR-G, U2 XC6222B331MR-G, U3 XC6222B331MR-G, U4 WM8960, U5 WM8960, U6 XC6222B331MR-G, U7 WM8960, U8 XC6222B331MR-G, U9 WM8960, Y1 24 MHz, Y2 24 MHz, Y3 24 MHz, Y4 24 MHz, Y5 24 MHz, Y6 24 MHz

Commit message: Production panel v10c
Parts:
- added AVDD-ISO10, AVDD-ISO11, AVDD-ISO6, AVDD-ISO7, AVDD-ISO8, AVDD-ISO9, LED10, LED11, LED6, LED7, LED8, LED9: (no value), SparkFun-Jumpers:SMT-JUMPER_2_NC_TRACE_SILK
- added C175, C176, C177, C197, C198, C204, C205, C206, C226, C227, C233, C234, C235, C255, C256, C262, C263, C264, C284, C285, C291, C292, C293, C313, C314, C320, C321, C322, C342, C343: 0.1uF, SparkFun-Capacitors:0402-TIGHT
- added C178, C179, C207, C208, C236, C237, C265, C266, C294, C295, C323, C324: 4.7uF, SparkFun-Capacitors:0402-TIGHT
- added C180, C209, C238, C267, C296, C325: 10nF, SparkFun-Capacitors:0402-TIGHT
- added C181, C182, C183, C184, C210, C211, C212, C213, C239, C240, C241, C242, C268, C269, C270, C271, C297, C298, C299, C300, C326, C327, C328, C329: 1nF, SparkFun-Capacitors:0402
- added C185, C186, C189, C190, C191, C192, C201, C214, C215, C218, C219, C220, C221, C230, C243, C244, C247, C248, C249, C250, C259, C272, C273, C276, C277, C278, C279, C288, C301, C302, C305, C306, C307, C308, C317, C330, C331, C334, C335, C336, C337, C346: 1.0uF, SparkFun-Capacitors:0402-TIGHT
- added C187, C188, C193, C194, C195, C196, C216, C217, C222, C223, C224, C225, C245, C246, C251, C252, C253, C254, C274, C275, C280, C281, C282, C283, C303, C304, C309, C310, C311, C312, C332, C333, C338, C339, C340, C341: 47nF, SparkFun-Capacitors:0402-TIGHT
- added C199, C200, C228, C229, C257, C258, C286, C287, C315, C316, C344, C345: 4.7uF, SparkFun-Capacitors:0603
- added C202, C203, C231, C232, C260, C261, C289, C290, C318, C319, C347, C348: 10uF, SparkFun-Capacitors:0402-TIGHT
- added D10, D11, D12, D7, D8, D9: RED, SparkFun-LED:LED-0603
- added FD25, FD26, FD27, FD28, FD29, FD30, FD31, FD32, FD33, FD34, FD35, FD36, FD37, FD38, FD39, FD40, FD41, FD42, FD43, FD44, FD45, FD46, FD47, FD48: FIDUCIALUFIDUCIAL, SparkFun-Aesthetics:FIDUCIAL-MICRO
- added I2C10, I2C11, I2C6, I2C7, I2C8, I2C9: JUMPER-SMT_3_2-NC_TRACE_SILK, SparkFun-Jumpers:SMT-JUMPER_3_2-NC_TRACE_SILK
- added J19, J22, J25, J28, J31, J34: QWIIC, SparkFun-Connectors:JST04_1MM_RA
- added J20, J21, J23, J24, J26, J27, J29, J30, J32, J33, J35, J36: (no value), SparkFun-Connectors:1X16_NO_SILK
- added L25, L26, L27, L28, L29, L30, L31, L32, L33, L34, L35, L36, L37, L38, L39, L40, L41, L42, L43, L44, L45, L46, L47, L48: 220Ω, SparkFun-Coils:0805
- added LOGO19, LOGO22, LOGO25, LOGO28, LOGO31, LOGO34: QWIIC_LOGO_4MM, SparkFun-Aesthetics:QWIIC_4MM
- added LOGO20, LOGO23, LOGO26, LOGO29, LOGO32, LOGO35: OSHW-LOGOS, SparkFun-Aesthetics:OSHW-LOGO-S
- added LOGO21, LOGO24, LOGO27, LOGO30, LOGO33, LOGO36: SFE_LOGO_NAME_FLAME.1_INCH, SparkFun-Aesthetics:SFE_LOGO_NAME_FLAME_.1
- added R100, R101, R102, R103, R104, R105, R116, R117, R118, R119, R120, R121, R132, R133, R134, R135, R136, R137, R148, R149, R150, R151, R152, R153, R164, R165, R166, R167, R168, R169, R180, R181, R182, R183, R184, R185: 100, SparkFun-Resistors:0402-TIGHT
- added R106, R107, R108, R109, R110, R112, R122, R123, R124, R125, R126, R128, R138, R139, R140, R141, R142, R144, R154, R155, R156, R157, R158, R160, R170, R171, R172, R173, R174, R176, R186, R187, R188, R189, R190, R192: 10Ω, SparkFun-Resistors:0402-TIGHT
- added R111, R127, R143, R159, R175, R191: 100k, SparkFun-Resistors:0402-TIGHT
- added R113, R114, R129, R130, R145, R146, R161, R162, R177, R178, R97, R98: 2.2k, SparkFun-Resistors:0402-TIGHT
- added R115, R131, R147, R163, R179, R99: 1k, SparkFun-Resistors:0402-TIGHT
- added SPKVDD10, SPKVDD11, SPKVDD6, SPKVDD7, SPKVDD8, SPKVDD9: (no value), SparkFun-Jumpers:SMT-JUMPER_3_1-NC_TRACE_SILK
- added U$463, U$540, U$617, U$694, U$771, U$848: (no value), output:#SR##4
- added U$464, U$541, U$618, U$695, U$772, U$849: (no value), output:#SR##5
- added U$465, U$542, U$619, U$696, U$773, U$850: (no value), output:#SL##6
- added U$466, U$543, U$620, U$697, U$774, U$851: (no value), output:#SL##7
- added U$467, U$478, U$498, U$499, U$500, U$502, U$503, U$504, U$505, U$506, U$508, U$509, U$544, U$555, U$575, U$576, U$577, U$579, U$580, U$581, U$582, U$583, U$585, U$586, U$621, U$632, U$652, U$653, U$654, U$656, U$657, U$658, U$659, U$660, U$662, U$663, U$698, U$709, U$729, U$730, U$731, U$733, U$734, U$735, U$736, U$737, U$739, U$740, U$775, U$786, U$806, U$807, U$808, U$810, U$811, U$812, U$813, U$814, U$816, U$817, U$852, U$863, U$883, U$884, U$885, U$887, U$888, U$889, U$890, U$891, U$893, U$894: (no value), output:#GND#8
- added U$468, U$545, U$622, U$699, U$776, U$853: (no value), output:#HPL#10
- added U$469, U$546, U$623, U$700, U$777, U$854: (no value), output:#HPR#11
- added U$470, U$479, U$547, U$556, U$624, U$633, U$701, U$710, U$778, U$787, U$855, U$864: (no value), output:#3V3#12
- added U$471, U$548, U$625, U$702, U$779, U$856: (no value), SparkFun-Aesthetics:SFE_LOGO_FLAME_.1
- added U$472, U$549, U$626, U$703, U$780, U$857: (no value), output:PWR12
- added U$473, U$550, U$627, U$704, U$781, U$858: (no value), output:#LED#17
- added U$474, U$551, U$628, U$705, U$782, U$859: (no value), output:#I2C#18
- added U$475, U$476, U$552, U$553, U$629, U$630, U$706, U$707, U$783, U$784, U$860, U$861: (no value), output:#VIN#19
- added U$477, U$501, U$554, U$578, U$631, U$655, U$708, U$732, U$785, U$809, U$862, U$886: (no value), output:#AVDD#22
- added U$480, U$557, U$634, U$711, U$788, U$865: (no value), output:#MICB#31
- added U$481, U$558, U$635, U$712, U$789, U$866: (no value), output:WM89600
- added U$482, U$559, U$636, U$713, U$790, U$867: (no value), output:AUDIO0
- added U$483, U$560, U$637, U$714, U$791, U$868: (no value), output:#SCL#40
- added U$484, U$561, U$638, U$715, U$792, U$869: (no value), output:#SDA#41
- added U$485, U$562, U$639, U$716, U$793, U$870: (no value), output:#MICBIAS#42
- added U$486, U$563, U$640, U$717, U$794, U$871: (no value), output:#HPL#43
- added U$487, U$564, U$641, U$718, U$795, U$872: (no value), output:#HPR#45
- added U$488, U$565, U$642, U$719, U$796, U$873: (no value), output:#SPK_LP#46
- added U$489, U$566, U$643, U$720, U$797, U$874: (no value), output:#SPK_LN#47
- added U$490, U$567, U$644, U$721, U$798, U$875: (no value), output:#SPK_RP#48
- added U$491, U$568, U$645, U$722, U$799, U$876: (no value), output:#SPK_RN#49
- added U$492, U$507, U$569, U$584, U$646, U$661, U$723, U$738, U$800, U$815, U$877, U$892: (no value), output:#SPKVDD#51
- added U$493, U$570, U$647, U$724, U$801, U$878: (no value), output:WM8960896054
- added U$494, U$571, U$648, U$725, U$802, U$879: (no value), output:AUDIO8960896055
- added U$495, U$572, U$649, U$726, U$803, U$880: (no value), output:CODEC8960896056
- added U$496, U$573, U$650, U$727, U$804, U$881: (no value), output:CODEC8960896057
- added U$497, U$574, U$651, U$728, U$805, U$882: (no value), output:#OUT3#0
- added U$510, U$587, U$664, U$741, U$818, U$895: (no value), output:##EN##1
- added U$511, U$588, U$665, U$742, U$819, U$896: (no value), output:##EN##2
- added U$512, U$589, U$666, U$743, U$820, U$897: (no value), output:#OUT3#4
- added U$513, U$590, U$667, U$744, U$821, U$898: (no value), output:#RINPUT1#0
- added U$514, U$591, U$668, U$745, U$822, U$899: (no value), output:#RINPUT2#0
- added U$515, U$592, U$669, U$746, U$823, U$900: (no value), output:#RINPUT3#0
- added U$516, U$593, U$670, U$747, U$824, U$901: (no value), output:#LINPUT1#0
- added U$517, U$594, U$671, U$748, U$825, U$902: (no value), output:#LINPUT2#0
- added U$518, U$595, U$672, U$749, U$826, U$903: (no value), output:#LINPUT3#0
- added U$519, U$596, U$673, U$750, U$827, U$904: (no value), output:#AVDD#ISO#0
- added U$520, U$597, U$674, U$751, U$828, U$905: (no value), output:#3V3#0
- added U$521, U$598, U$675, U$752, U$829, U$906: (no value), output:#VIN#0
- added U$522, U$599, U$676, U$753, U$830, U$907: (no value), output:#SCL#0
- added U$523, U$600, U$677, U$754, U$831, U$908: (no value), output:#SDA#0
- added U$524, U$601, U$678, U$755, U$832, U$909: (no value), output:#RIN3#0
- added U$525, U$602, U$679, U$756, U$833, U$910: (no value), output:#RIN2#0
- added U$526, U$603, U$680, U$757, U$834, U$911: (no value), output:#RIN1#0
- added U$527, U$604, U$681, U$758, U$835, U$912: (no value), output:#LIN1#0
- added U$528, U$605, U$682, U$759, U$836, U$913: (no value), output:#LIN2#0
- added U$529, U$606, U$683, U$760, U$837, U$914: (no value), output:#LIN3#0
- added U$530, U$607, U$684, U$761, U$838, U$915: (no value), output:#BCLK#0
- added U$531, U$608, U$685, U$762, U$839, U$916: (no value), output:#ALRC#0
- added U$532, U$609, U$686, U$763, U$840, U$917: (no value), output:#DLRC#1
- added U$533, U$610, U$687, U$764, U$841, U$918: (no value), output:#ADCLRC#2
- added U$534, U$611, U$688, U$765, U$842, U$919: (no value), output:#DACLRC#4
- added U$535, U$612, U$689, U$766, U$843, U$920: (no value), output:#BCLK#5
- added U$536, U$613, U$690, U$767, U$844, U$921: (no value), output:#ADCDAT#6
- added U$537, U$614, U$691, U$768, U$845, U$922: (no value), output:#DACDAT#8
- added U$538, U$615, U$692, U$769, U$846, U$923: (no value), output:#DDAT#9
- added U$539, U$616, U$693, U$770, U$847, U$924: (no value), output:#ADAT#10
- added U13, U15, U17, U19, U21, U23: WM8960, SparkFun-IC-Special-Function:QFN-32
- added U14, U16, U18, U20, U22, U24: XC6222B331MR-G, SparkFun-IC-Power:SOT23-5
- added Y10, Y11, Y12, Y7, Y8, Y9: 24 MHz, SparkFun-Clocks:RESONATOR-SMD-3.2X2.5
- U$100, U$177, U$254, U$331, U$408: device output:WM89600 -> output:#MICBIAS#42
- U$101, U$178, U$255, U$332, U$409: device output:AUDIO0 -> output:#HPL#43
- U$102, U$179, U$256, U$333, U$410: device output:#BCLK#35 -> output:#HPR#45
- U$103, U$180, U$257, U$334, U$411: device output:#DACLRC#36 -> output:#SPK_LP#46
- U$104, U$181, U$258, U$335, U$412: device output:#DACDAT#37 -> output:#SPK_LN#47
- U$105, U$182, U$259, U$336, U$413: device output:#ADCLRC#38 -> output:#SPK_RP#48
- U$106, U$183, U$260, U$337, U$414: device output:#ADCDAT#39 -> output:#SPK_RN#49
- U$107, U$184, U$261, U$338, U$415: device output:#SCL#40 -> output:#SPKVDD#51
- U$108, U$185, U$262, U$339, U$416: device output:#SDA#41 -> output:WM8960896054
- U$109, U$186, U$263, U$340, U$417: device output:#MICBIAS#42 -> output:AUDIO8960896055
- U$110, U$187, U$264, U$341, U$418: device output:#HPL#43 -> output:CODEC8960896056
- U$111, U$188, U$265, U$342, U$419: device output:#HPR#45 -> output:CODEC8960896057
- U$112, U$189, U$266, U$343, U$420: device output:#SPK_LP#46 -> output:#OUT3#0
- U$113, U$190, U$267, U$344, U$421: device output:#SPK_LN#47 -> output:#GND#8
- U$114, U$191, U$268, U$345, U$422: device output:#SPK_RP#48 -> output:#GND#8
- U$115, U$192, U$269, U$346, U$423: device output:#SPK_RN#49 -> output:#GND#8
- U$116, U$193, U$270, U$347, U$424: device output:#SPKVDD#51 -> output:#AVDD#22
- U$117, U$194, U$271, U$348, U$425: device output:WM8960896054 -> output:#GND#8
- U$118, U$195, U$272, U$349, U$426: device output:AUDIO8960896055 -> output:#GND#8
- U$119, U$196, U$273, U$350, U$427: device output:CODEC8960896056 -> output:#GND#8
- U$120, U$197, U$274, U$351, U$428: device output:CODEC8960896057 -> output:#GND#8
- U$121, U$198, U$275, U$352, U$429: device output:#OUT3#0 -> output:#GND#8
- U$122, U$199, U$276, U$353, U$430: device output:#GND#8 -> output:#SPKVDD#51
- U$125, U$202, U$279, U$356, U$433: device output:#AVDD#22 -> output:##EN##1
- U$126, U$203, U$280, U$357, U$434: device output:#GND#8 -> output:##EN##2
- U$127, U$204, U$281, U$358, U$435: device output:#GND#8 -> output:#OUT3#4
- U$128, U$205, U$282, U$359, U$436: device output:#GND#8 -> output:#RINPUT1#0
- U$129, U$206, U$283, U$360, U$437: device output:#GND#8 -> output:#RINPUT2#0
- U$130, U$207, U$284, U$361, U$438: device output:#GND#8 -> output:#RINPUT3#0
- U$131, U$208, U$285, U$362, U$439: device output:#SPKVDD#51 -> output:#LINPUT1#0
- U$132, U$209, U$286, U$363, U$440: device output:#GND#8 -> output:#LINPUT2#0
- U$133, U$210, U$287, U$364, U$441: device output:#GND#8 -> output:#LINPUT3#0
- U$134, U$211, U$288, U$365, U$442: device output:##EN##1 -> output:#AVDD#ISO#0
- U$135, U$212, U$289, U$366, U$443: device output:##EN##2 -> output:#3V3#0
- U$136, U$213, U$290, U$367, U$444: device output:#OUT3#4 -> output:#VIN#0
- U$137, U$214, U$291, U$368, U$445: device output:#RINPUT1#0 -> output:#SCL#0
- U$138, U$215, U$292, U$369, U$446: device output:#RINPUT2#0 -> output:#SDA#0
- U$139, U$216, U$293, U$370, U$447: device output:#RINPUT3#0 -> output:#RIN3#0
- U$140, U$217, U$294, U$371, U$448: device output:#LINPUT1#0 -> output:#RIN2#0
- U$141, U$218, U$295, U$372, U$449: device output:#LINPUT2#0 -> output:#RIN1#0
- U$142, U$219, U$296, U$373, U$450: device output:#LINPUT3#0 -> output:#LIN1#0
- U$143, U$220, U$297, U$374, U$451: device output:#AVDD#ISO#0 -> output:#LIN2#0
- U$144, U$221, U$298, U$375, U$452: device output:#3V3#0 -> output:#LIN3#0
- U$145, U$222, U$299, U$376, U$453: device output:#VIN#0 -> output:#BCLK#0
- U$146, U$223, U$300, U$377, U$454: device output:#SCL#0 -> output:#ALRC#0
- U$147, U$224, U$301, U$378, U$455: device output:#SDA#0 -> output:#DLRC#1
- U$148, U$225, U$302, U$379, U$456: device output:#ADAT#0 -> output:#ADCLRC#2
- U$149, U$226, U$303, U$380, U$457: device output:#RIN3#0 -> output:#DACLRC#4
- U$150, U$227, U$304, U$381, U$458: device output:#RIN2#0 -> output:#BCLK#5
- U$151, U$228, U$305, U$382, U$459: device output:#RIN1#0 -> output:#ADCDAT#6
- U$152, U$229, U$306, U$383, U$460: device output:#LIN1#0 -> output:#DACDAT#8
- U$153, U$230, U$307, U$384, U$461: device output:#LIN2#0 -> output:#DDAT#9
- U$154, U$231, U$308, U$385, U$462: device output:#LIN3#0 -> output:#ADAT#10
- U$172, U$249, U$326, U$403, U$95: device output:#BC#24 -> output:#MICB#31
- U$173, U$250, U$327, U$404, U$96: device output:#DLRC#25 -> output:WM89600
- U$174, U$251, U$328, U$405, U$97: device output:#ALR#29 -> output:AUDIO0
- U$175, U$252, U$329, U$406, U$98: device output:#DDT#30 -> output:#SCL#40
- U$176, U$253, U$330, U$407, U$99: device output:#MICB#31 -> output:#SDA#41
- U$23: device output:#SL##6 -> output:#ALRC#0
- U$24: device output:#SL##7 -> output:#DLRC#1
- U$25: device output:#GND#8 -> output:#SR##5
- U$33: device output:#HPL#10 -> output:#SL##6
- U$42: device output:#HPR#11 -> output:#SL##7
- U$43: device output:#3V3#12 -> output:#GND#8
- U$5: device output:#SR##4 -> output:#BCLK#0
- U$52: device output:#BC#24 -> output:#ADCLRC#2
- U$53: device output:#DLRC#25 -> output:#HPL#10
- U$55: device output:#ADAT#0 -> output:#DACLRC#4
- U$57: device output:#ALR#29 -> output:#BCLK#5
- U$58: device output:#DDT#30 -> output:#ADCDAT#6
- U$6: device output:#SR##5 -> output:#SR##4
- U$69: device output:#BCLK#35 -> output:#DDAT#9
- U$70: device output:#DACLRC#36 -> output:#DACDAT#8
- U$71: device output:#DACDAT#37 -> output:#ADAT#10
- U$72: device output:#ADCLRC#38 -> output:#HPR#11
- U$73: device output:#ADCDAT#39 -> output:#3V3#12
- moved E$1 82.3 mm to (6.86, 166.2)
- moved E$2 82.3 mm to (6.86, 166.2)
- moved E$3 82.3 mm to (70.3, 166.2)
- moved E$4 82.3 mm to (70.3, 166.2)
- moved U$5 54.8 mm to (4.19, 36.8)
- moved U$24 50.5 mm to (4.24, 34.3)
- moved U$23 49.3 mm to (4.32, 29.2)
- moved U$53 46.1 mm to (47.7, 19.0)
- moved U$72 45.1 mm to (47.7, 13.9), flipped to the top
- moved U$355 42.0 mm to (47.4, 80.5), flipped to the top
- moved U$124 42.0 mm to (47.4, 39.4), flipped to the top
- moved U$278 42.0 mm to (21.5, 80.5), flipped to the top
- moved U$432 42.0 mm to (73.3, 80.5), flipped to the top
- moved U$201 42.0 mm to (73.3, 39.4), flipped to the top
- moved U$277 38.1 mm to (3.87, 80.5)
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Connections:
- new net 3.3V10: C291.2, C292.2, C293.2, C296.1, I2C10.2, J31.2, J32.8, LED10.2, SPKVDD10.1, U21.10, U21.8, Y11.1, Y11.4
- new net 3.3V11: C320.2, C321.2, C322.2, C325.1, I2C11.2, J34.2, J35.8, LED11.2, SPKVDD11.1, U23.10, U23.8, Y12.1, Y12.4
- new net 3.3V6: C175.2, C176.2, C177.2, C180.1, I2C6.2, J19.2, J20.8, LED6.2, SPKVDD6.1, U13.10, U13.8, Y7.1, Y7.4
- new net 3.3V7: C204.2, C205.2, C206.2, C209.1, I2C7.2, J22.2, J23.8, LED7.2, SPKVDD7.1, U15.10, U15.8, Y8.1, Y8.4
- new net 3.3V8: C233.2, C234.2, C235.2, C238.1, I2C8.2, J25.2, J26.8, LED8.2, SPKVDD8.1, U17.10, U17.8, Y9.1, Y9.4
- new net 3.3V9: C262.2, C263.2, C264.2, C267.1, I2C9.2, J28.2, J29.8, LED9.2, SPKVDD9.1, U19.10, U19.8, Y10.1, Y10.4
- new net ADCDAT10: J32.11, R173.1
- new net ADCDAT11: J35.11, R189.1
- new net ADCDAT6: J20.11, R109.1
- new net ADCDAT7: J23.11, R125.1
- new net ADCDAT8: J26.11, R141.1
- new net ADCDAT9: J29.11, R157.1
- new net ADCLRC10: J32.12, R170.1
- new net ADCLRC11: J35.12, R186.1
- new net ADCLRC6: J20.12, R106.1
- new net ADCLRC7: J23.12, R122.1
- new net ADCLRC8: J26.12, R138.1
- new net ADCLRC9: J29.12, R154.1
- new net AVDD-REG10: AVDD-ISO10.1, C317.1, C318.1, U22.5
- new net AVDD-REG11: AVDD-ISO11.1, C346.1, C347.1, U24.5
- new net AVDD-REG6: AVDD-ISO6.1, C201.1, C202.1, U14.5
- new net AVDD-REG7: AVDD-ISO7.1, C230.1, C231.1, U16.5
- new net AVDD-REG8: AVDD-ISO8.1, C259.1, C260.1, U18.5
- new net AVDD-REG9: AVDD-ISO9.1, C288.1, C289.1, U20.5
- new net AVDD10: AVDD-ISO10.2, C314.2, J33.5, U21.32
- new net AVDD11: AVDD-ISO11.2, C343.2, J36.5, U23.32
- new net AVDD6: AVDD-ISO6.2, C198.2, J21.5, U13.32
- new net AVDD7: AVDD-ISO7.2, C227.2, J24.5, U15.32
- new net AVDD8: AVDD-ISO8.2, C256.2, J27.5, U17.32
- new net AVDD9: AVDD-ISO9.2, C285.2, J30.5, U19.32
- new net BCLK10: J32.15, R172.1
- new net BCLK11: J35.15, R188.1
- new net BCLK6: J20.15, R108.1
- new net BCLK7: J23.15, R124.1
- new net BCLK8: J26.15, R140.1
- new net BCLK9: J29.15, R156.1
- new net DACDAT10: J32.13, R174.1
- new net DACDAT11: J35.13, R190.1
- new net DACDAT6: J20.13, R110.1
- new net DACDAT7: J23.13, R126.1
- new net DACDAT8: J26.13, R142.1
- new net DACDAT9: J29.13, R158.1
- new net DACLRC10: J32.14, R171.1
- new net DACLRC11: J35.14, R187.1
- new net DACLRC6: J20.14, R107.1
- new net DACLRC7: J23.14, R123.1
- new net DACLRC8: J26.14, R139.1
- new net DACLRC9: J29.14, R155.1
- new net EN10: J32.3, R175.2, U22.3
- new net EN11: J35.3, R191.2, U24.3
- new net EN6: J20.3, R111.2, U14.3
- new net EN7: J23.3, R127.2, U16.3
- new net EN8: J26.3, R143.2, U18.3
- new net EN9: J29.3, R159.2, U20.3
- new net GND10: C291.1, C292.1, C293.1, C294.1, C295.1, C296.2, C297.2, C298.2, C299.2, C300.2, C303.2, C304.2, C309.2, C310.2, C311.2, C312.2, C313.2, C314.1, C315.2, C316.2, C317.2, C318.2, C319.2, J31.1, J32.1, J32.16, J32.2, J32.6, J32.7, J33.16, R163.1, U21.20, U21.24, U21.28, U21.9, U21.PADDLE, U22.2, Y11.2
- new net GND11: C320.1, C321.1, C322.1, C323.1, C324.1, C325.2, C326.2, C327.2, C328.2, C329.2, C332.2, C333.2, C338.2, C339.2, C340.2, C341.2, C342.2, C343.1, C344.2, C345.2, C346.2, C347.2, C348.2, J34.1, J35.1, J35.16, J35.2, J35.6, J35.7, J36.16, R179.1, U23.20, U23.24, U23.28, U23.9, U23.PADDLE, U24.2, Y12.2
- new net GND6: C175.1, C176.1, C177.1, C178.1, C179.1, C180.2, C181.2, C182.2, C183.2, C184.2, C187.2, C188.2, C193.2, C194.2, C195.2, C196.2, C197.2, C198.1, C199.2, C200.2, C201.2, C202.2, C203.2, J19.1, J20.1, J20.16, J20.2, J20.6, J20.7, J21.16, R99.1, U13.20, U13.24, U13.28, U13.9, U13.PADDLE, U14.2, Y7.2
- new net GND7: C204.1, C205.1, C206.1, C207.1, C208.1, C209.2, C210.2, C211.2, C212.2, C213.2, C216.2, C217.2, C222.2, C223.2, C224.2, C225.2, C226.2, C227.1, C228.2, C229.2, C230.2, C231.2, C232.2, J22.1, J23.1, J23.16, J23.2, J23.6, J23.7, J24.16, R115.1, U15.20, U15.24, U15.28, U15.9, U15.PADDLE, U16.2, Y8.2
- new net GND8: C233.1, C234.1, C235.1, C236.1, C237.1, C238.2, C239.2, C240.2, C241.2, C242.2, C245.2, C246.2, C251.2, C252.2, C253.2, C254.2, C255.2, C256.1, C257.2, C258.2, C259.2, C260.2, C261.2, J25.1, J26.1, J26.16, J26.2, J26.6, J26.7, J27.16, R131.1, U17.20, U17.24, U17.28, U17.9, U17.PADDLE, U18.2, Y9.2
- new net GND9: C262.1, C263.1, C264.1, C265.1, C266.1, C267.2, C268.2, C269.2, C270.2, C271.2, C274.2, C275.2, C280.2, C281.2, C282.2, C283.2, C284.2, C285.1, C286.2, C287.2, C288.2, C289.2, C290.2, J28.1, J29.1, J29.16, J29.2, J29.6, J29.7, J30.16, R147.1, U19.20, U19.24, U19.28, U19.9, U19.PADDLE, U20.2, Y10.2
- new net HP_L10: J33.8, U21.31
- new net HP_L11: J36.8, U23.31
- new net HP_L6: J21.8, U13.31
- new net HP_L7: J24.8, U15.31
- new net HP_L8: J27.8, U17.31
- new net HP_L9: J30.8, U19.31
- new net HP_R10: J33.6, U21.29
- new net HP_R11: J36.6, U23.29
- new net HP_R6: J21.6, U13.29
- new net HP_R7: J24.6, U15.29
- new net HP_R8: J27.6, U17.29
- new net HP_R9: J30.6, U19.29
- new net LINPUT19: J21.12, R100.1
- new net LINPUT20: J21.10, R102.1
- new net LINPUT21: J21.11, R101.1
- new net LINPUT22: J24.12, R116.1
- new net LINPUT23: J24.10, R118.1
- new net LINPUT24: J24.11, R117.1
- new net LINPUT25: J27.12, R132.1
- new net LINPUT26: J27.10, R134.1
- new net LINPUT27: J27.11, R133.1
- new net LINPUT28: J30.12, R148.1
- new net LINPUT29: J30.10, R150.1
- new net LINPUT30: J30.11, R149.1
- new net LINPUT31: J33.12, R164.1
- new net LINPUT32: J33.10, R166.1
- new net LINPUT33: J33.11, R165.1
- new net LINPUT34: J36.12, R180.1
- new net LINPUT35: J36.10, R182.1
- new net LINPUT36: J36.11, R181.1
- new net MICBIAS10: C295.2, J33.9, U21.1
- new net MICBIAS11: C324.2, J36.9, U23.1
- new net MICBIAS6: C179.2, J21.9, U13.1
- new net MICBIAS7: C208.2, J24.9, U15.1
- new net MICBIAS8: C237.2, J27.9, U17.1
- new net MICBIAS9: C266.2, J30.9, U19.1
- new net N$169: C185.2, U13.4
- new net N$170: C190.2, U13.5
- new net N$171: C178.2, U13.27
- new net N$172: I2C6.3, R97.2
- new net N$173: I2C6.1, R98.2
- new net N$174: R112.1, Y7.3
- new net N$175: C192.2, U13.7
- new net N$176: C191.2, U13.6
- new net N$177: C189.2, U13.2
- new net N$178: C186.2, U13.3
- new net N$179: L27.1, U13.22
- new net N$180: L28.1, U13.19
- new net N$181: L26.1, U13.25
- new net N$182: L25.1, U13.23
- new net N$183: D7.C, R99.2
- new net N$184: C186.1, C187.1, R101.2
- new net N$185: C185.1, C188.1, R100.2
- new net N$186: C189.1, C193.1, R102.2
- new net N$187: C190.1, C194.1, R103.2
- new net N$188: C191.1, C195.1, R104.2
- new net N$189: C192.1, C196.1, R105.2
- new net N$190: R106.2, U13.15
- new net N$191: R107.2, U13.13
- new net N$192: R108.2, U13.12
- new net N$193: R109.2, U13.16
- new net N$194: R110.2, U13.14
- new net N$195: R112.2, U13.11
- new net N$196: D7.A, LED6.1
- new net N$197: C214.2, U15.4
- new net N$198: C219.2, U15.5
- new net N$199: C207.2, U15.27
- new net N$200: I2C7.3, R113.2
- new net N$201: I2C7.1, R114.2
- new net N$202: R128.1, Y8.3
- new net N$203: C221.2, U15.7
- new net N$204: C220.2, U15.6
- new net N$205: C218.2, U15.2
- new net N$206: C215.2, U15.3
- new net N$207: L31.1, U15.22
- new net N$208: L32.1, U15.19
- new net N$209: L30.1, U15.25
- new net N$210: L29.1, U15.23
- new net N$211: D8.C, R115.2
- new net N$212: C215.1, C216.1, R117.2
- new net N$213: C214.1, C217.1, R116.2
- new net N$214: C218.1, C222.1, R118.2
- new net N$215: C219.1, C223.1, R119.2
- new net N$216: C220.1, C224.1, R120.2
- new net N$217: C221.1, C225.1, R121.2
- new net N$218: R122.2, U15.15
- new net N$219: R123.2, U15.13
- new net N$220: R124.2, U15.12
- new net N$221: R125.2, U15.16
- new net N$222: R126.2, U15.14
- new net N$223: R128.2, U15.11
- new net N$224: D8.A, LED7.1
- new net N$225: C243.2, U17.4
- new net N$226: C248.2, U17.5
- new net N$227: C236.2, U17.27
- new net N$228: I2C8.3, R129.2
- new net N$229: I2C8.1, R130.2
- new net N$230: R144.1, Y9.3
- new net N$231: C250.2, U17.7
- new net N$232: C249.2, U17.6
- new net N$233: C247.2, U17.2
- new net N$234: C244.2, U17.3
- new net N$235: L35.1, U17.22
- new net N$236: L36.1, U17.19
- new net N$237: L34.1, U17.25
- new net N$238: L33.1, U17.23
- new net N$239: D9.C, R131.2
- new net N$240: C244.1, C245.1, R133.2
- new net N$241: C243.1, C246.1, R132.2
- new net N$242: C247.1, C251.1, R134.2
- new net N$243: C248.1, C252.1, R135.2
- new net N$244: C249.1, C253.1, R136.2
- new net N$245: C250.1, C254.1, R137.2
- new net N$246: R138.2, U17.15
- new net N$247: R139.2, U17.13
- new net N$248: R140.2, U17.12
- new net N$249: R141.2, U17.16
- new net N$250: R142.2, U17.14
- new net N$251: R144.2, U17.11
- new net N$252: D9.A, LED8.1
- new net N$253: C272.2, U19.4
- new net N$254: C277.2, U19.5
- new net N$255: C265.2, U19.27
- new net N$256: I2C9.3, R145.2
- new net N$257: I2C9.1, R146.2
- new net N$258: R160.1, Y10.3
- new net N$259: C279.2, U19.7
- new net N$260: C278.2, U19.6
- new net N$261: C276.2, U19.2
- new net N$262: C273.2, U19.3
- new net N$263: L39.1, U19.22
- new net N$264: L40.1, U19.19
- new net N$265: L38.1, U19.25
- new net N$266: L37.1, U19.23
- new net N$267: D10.C, R147.2
- new net N$268: C273.1, C274.1, R149.2
- new net N$269: C272.1, C275.1, R148.2
- new net N$270: C276.1, C280.1, R150.2
- new net N$271: C277.1, C281.1, R151.2
- new net N$272: C278.1, C282.1, R152.2
- new net N$273: C279.1, C283.1, R153.2
- new net N$274: R154.2, U19.15
- new net N$275: R155.2, U19.13
- new net N$276: R156.2, U19.12
- new net N$277: R157.2, U19.16
- new net N$278: R158.2, U19.14
- new net N$279: R160.2, U19.11
- new net N$280: D10.A, LED9.1
- new net N$281: C301.2, U21.4
- new net N$282: C306.2, U21.5
- new net N$283: C294.2, U21.27
- new net N$284: I2C10.3, R161.2
- new net N$285: I2C10.1, R162.2
- new net N$286: R176.1, Y11.3
- new net N$287: C308.2, U21.7
- new net N$288: C307.2, U21.6
- new net N$289: C305.2, U21.2
- new net N$290: C302.2, U21.3
- new net N$291: L43.1, U21.22
- new net N$292: L44.1, U21.19
- new net N$293: L42.1, U21.25
- new net N$294: L41.1, U21.23
- new net N$295: D11.C, R163.2
- new net N$296: C302.1, C303.1, R165.2
- new net N$297: C301.1, C304.1, R164.2
- new net N$298: C305.1, C309.1, R166.2
- new net N$299: C306.1, C310.1, R167.2
- new net N$300: C307.1, C311.1, R168.2
- new net N$301: C308.1, C312.1, R169.2
- new net N$302: R170.2, U21.15
- new net N$303: R171.2, U21.13
- new net N$304: R172.2, U21.12
- new net N$305: R173.2, U21.16
- new net N$306: R174.2, U21.14
- new net N$307: R176.2, U21.11
- new net N$308: D11.A, LED10.1
- new net N$309: C330.2, U23.4
- new net N$310: C335.2, U23.5
- new net N$311: C323.2, U23.27
- new net N$312: I2C11.3, R177.2
- new net N$313: I2C11.1, R178.2
- new net N$314: R192.1, Y12.3
- new net N$315: C337.2, U23.7
- new net N$316: C336.2, U23.6
- new net N$317: C334.2, U23.2
- new net N$318: C331.2, U23.3
- new net N$319: L47.1, U23.22
- new net N$320: L48.1, U23.19
- new net N$321: L46.1, U23.25
- new net N$322: L45.1, U23.23
- new net N$323: D12.C, R179.2
- new net N$324: C331.1, C332.1, R181.2
- new net N$325: C330.1, C333.1, R180.2
- new net N$326: C334.1, C338.1, R182.2
- new net N$327: C335.1, C339.1, R183.2
- new net N$328: C336.1, C340.1, R184.2
- new net N$329: C337.1, C341.1, R185.2
- new net N$330: R186.2, U23.15
- new net N$331: R187.2, U23.13
- new net N$332: R188.2, U23.12
- new net N$333: R189.2, U23.16
- new net N$334: R190.2, U23.14
- new net N$335: R192.2, U23.11
- new net N$336: D12.A, LED11.1
- new net OUT10: J30.7, U19.30
- new net OUT11: J33.7, U21.30
- new net OUT12: J36.7, U23.30
- new net OUT7: J21.7, U13.30
- new net OUT8: J24.7, U15.30
- new net OUT9: J27.7, U17.30
- new net RINPUT19: J21.13, R103.1
- new net RINPUT20: J21.15, R105.1
- new net RINPUT21: J21.14, R104.1
- new net RINPUT22: J24.13, R119.1
- new net RINPUT23: J24.15, R121.1
- new net RINPUT24: J24.14, R120.1
- new net RINPUT25: J27.13, R135.1
- new net RINPUT26: J27.15, R137.1
- new net RINPUT27: J27.14, R136.1
- new net RINPUT28: J30.13, R151.1
- new net RINPUT29: J30.15, R153.1
- new net RINPUT30: J30.14, R152.1
- new net RINPUT31: J33.13, R167.1
- new net RINPUT32: J33.15, R169.1
- new net RINPUT33: J33.14, R168.1
- new net RINPUT34: J36.13, R183.1
- new net RINPUT35: J36.15, R185.1
- new net RINPUT36: J36.14, R184.1
- new net SCL10: J31.4, J32.10, R161.1, U21.17
- new net SCL11: J34.4, J35.10, R177.1, U23.17
- new net SCL6: J19.4, J20.10, R97.1, U13.17
- new net SCL7: J22.4, J23.10, R113.1, U15.17
- new net SCL8: J25.4, J26.10, R129.1, U17.17
- new net SCL9: J28.4, J29.10, R145.1, U19.17
- new net SDA10: J31.3, J32.9, R162.1, U21.18
- new net SDA11: J34.3, J35.9, R178.1, U23.18
- new net SDA6: J19.3, J20.9, R98.1, U13.18
- new net SDA7: J22.3, J23.9, R114.1, U15.18
- new net SDA8: J25.3, J26.9, R130.1, U17.18
- new net SDA9: J28.3, J29.9, R146.1, U19.18
- new net SPKVDD10: C315.1, C316.1, J32.5, SPKVDD10.2, U21.21, U21.26
- new net SPKVDD11: C344.1, C345.1, J35.5, SPKVDD11.2, U23.21, U23.26
- new net SPKVDD6: C199.1, C200.1, J20.5, SPKVDD6.2, U13.21, U13.26
- new net SPKVDD7: C228.1, C229.1, J23.5, SPKVDD7.2, U15.21, U15.26
- new net SPKVDD8: C257.1, C258.1, J26.5, SPKVDD8.2, U17.21, U17.26
- new net SPKVDD9: C286.1, C287.1, J29.5, SPKVDD9.2, U19.21, U19.26
- new net SPK_LN10: C297.1, J33.3, L41.2
- new net SPK_LN11: C326.1, J36.3, L45.2
- new net SPK_LN6: C181.1, J21.3, L25.2
- new net SPK_LN7: C210.1, J24.3, L29.2
- new net SPK_LN8: C239.1, J27.3, L33.2
- new net SPK_LN9: C268.1, J30.3, L37.2
- new net SPK_LP10: C298.1, J33.4, L42.2
- new net SPK_LP11: C327.1, J36.4, L46.2
- new net SPK_LP6: C182.1, J21.4, L26.2
- new net SPK_LP7: C211.1, J24.4, L30.2
- new net SPK_LP8: C240.1, J27.4, L34.2
- new net SPK_LP9: C269.1, J30.4, L38.2
- new net SPK_RN10: C300.1, J33.1, L44.2
- new net SPK_RN11: C329.1, J36.1, L48.2
- new net SPK_RN6: C184.1, J21.1, L28.2
- new net SPK_RN7: C213.1, J24.1, L32.2
- new net SPK_RN8: C242.1, J27.1, L36.2
- new net SPK_RN9: C271.1, J30.1, L40.2
- new net SPK_RP10: C299.1, J33.2, L43.2
- new net SPK_RP11: C328.1, J36.2, L47.2
- new net SPK_RP6: C183.1, J21.2, L27.2
- new net SPK_RP7: C212.1, J24.2, L31.2
- new net SPK_RP8: C241.1, J27.2, L35.2
- new net SPK_RP9: C270.1, J30.2, L39.2
- new net VIN10: C313.1, C319.1, J32.4, R175.1, SPKVDD10.3, U22.1
- new net VIN11: C342.1, C348.1, J35.4, R191.1, SPKVDD11.3, U24.1
- new net VIN6: C197.1, C203.1, J20.4, R111.1, SPKVDD6.3, U14.1
- new net VIN7: C226.1, C232.1, J23.4, R127.1, SPKVDD7.3, U16.1
- new net VIN8: C255.1, C261.1, J26.4, R143.1, SPKVDD8.3, U18.1
- new net VIN9: C284.1, C290.1, J29.4, R159.1, SPKVDD9.3, U20.1
Routing:
- net GND11: track 0.00 -> 43.9 mm, vias 0 -> 63
- net GND9: track 0.00 -> 43.9 mm, vias 0 -> 63
- net GND10: track 0.00 -> 43.9 mm, vias 0 -> 63
- net GND6: track 0.00 -> 43.9 mm, vias 0 -> 63
- net GND8: track 0.00 -> 43.9 mm, vias 0 -> 63
- net GND7: track 0.00 -> 43.9 mm, vias 0 -> 63
- net SCL9: track 0.00 -> 38.7 mm, vias 0 -> 4
- net SCL8: track 0.00 -> 38.7 mm, vias 0 -> 4
- net SCL11: track 0.00 -> 38.7 mm, vias 0 -> 4
- net SCL10: track 0.00 -> 38.7 mm, vias 0 -> 4
- net SCL7: track 0.00 -> 38.7 mm, vias 0 -> 4
- net SCL6: track 0.00 -> 38.7 mm, vias 0 -> 4
- net SDA11: track 0.00 -> 34.1 mm, vias 0 -> 2
- net SDA9: track 0.00 -> 34.1 mm, vias 0 -> 2
- net SDA10: track 0.00 -> 34.1 mm, vias 0 -> 2
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- added copper zone on layer 15, net 3.3V10
- added copper zone on layer 15, net 3.3V11
- added copper zone on layer 15, net 3.3V6
- added copper zone on layer 15, net 3.3V7
- added copper zone on layer 15, net 3.3V8
- added copper zone on layer 15, net 3.3V9
- added copper zone on layer 15, net AVDD10
- added copper zone on layer 15, net AVDD11
- added copper zone on layer 15, net AVDD6
- added copper zone on layer 15, net AVDD7
- added copper zone on layer 15, net AVDD8
- added copper zone on layer 15, net AVDD9
- added copper zone on layer 16, net GND10
- added copper zone on layer 2, net GND10
- added copper zone on layer 16, net GND11
- added copper zone on layer 2, net GND11
- added copper zone on layer 16, net GND6
- added copper zone on layer 2, net GND6
- added copper zone on layer 16, net GND7
- added copper zone on layer 2, net GND7
- added copper zone on layer 16, net GND8
- added copper zone on layer 2, net GND8
- added copper zone on layer 16, net GND9
- added copper zone on layer 2, net GND9
Other:
- board size 97.3 x 96 mm -> 97.3 x 178.3 mm
- board text added: "v10"
- board text removed: "v01"
